File: PCB_Hardware/Cain/Cain_V1.0/CAN2.0.kicad_sch (KiCad schematic)
At the start: 19 parts, among them J3 Conn_02x04_Odd_Even, J4 Conn_02x04_Odd_Even, U2 SN65HVD230DR-JSM

Commit message: File dump
Parts:
- C13, C14, C15: JLCPCB Part Number (none) -> C1525
- D1, D5: JLCPCB Part Number (none) -> C152727
- D3, D6: JLCPCB Part Number (none) -> C434419
- F1: JLCPCB Part Number (none) -> C75464
- F2: JLCPCB Part Number (none) -> C561584
- J3, J4: JLCPCB Part Number (none) -> C157975
- R12, R13: JLCPCB Part Number (none) -> C4109
- R3: JLCPCB Part Number (none) -> C1091
- TP2, TP4, TP5, TP9: now not fitted
- U2: JLCPCB Part Number (none) -> C46596299
Connections:
- net GND: no longer J4.3 (Pin_3)
- no-connect marks 0 -> 1
Other:
- note added: "CAN 2.0 / Power"
