File: PCB_Hardware/Cain/Cain_V1.0/Cain_V1.0.kicad_pcb (KiCad board)
At the start: 4 copper layers, 30 x 37 mm, 75 parts, among them J1 Conn_ARM_JTAG_SWD_10, J2 Conn_01x02_Socket, J3 Conn_02x04_Odd_Even, J4 Conn_02x04_Odd_Even, J5 Conn_01x04_Pin, J6 Conn_01x04_Pin, Q1 STN4NF03L, SW1 TSB008A2518A, U1 STM32F105RBT6, U2 SN65HVD230DR-JSM, U3 GZP168-102S, U4 INA333AIDRGR, U5 24LC01BH, U6 INA180A2IDBVR, Y1 X50328MSB2GI (8Mhz)

Commit message: File dump
Parts:
- added G***: LOGO, Tutor_Common_Parts:Tutor_Logo_Small, B.Cu at (144.6, 106.8)
- D3: footprint Diode_SMD:D_0603_1608Metric -> LED_SMD:LED_0603_1608Metric
- D6: value YELLOW -> RED; footprint Diode_SMD:D_0603_1608Metric -> LED_SMD:LED_0603_1608Metric
- D7: value LED -> RED
- H1, H2: footprint MountingHole:MountingHole_2.7mm_M2.5 -> MountingHole:MountingHole_3.2mm_M3
- U5: value 24LC01BH -> M24C01-RMN; footprint Package_TO_SOT_SMD:SC-70-8 -> Package_SO:SOIC-8_3.9x4.9mm_P1.27mm
- moved U5 4.63 mm to (147.0, 101.2)
- moved TP7 4.31 mm to (145.0, 107.4)
- moved TP6 3.84 mm to (142.4, 110.2)
- moved C21 3.54 mm to (151.4, 102.6)
- moved J5 3.00 mm to (139.4, 109.6), turned to 180 degrees
- moved C12 2.81 mm to (148.8, 97.8), turned to 0 degrees
- moved TP9 0.43 mm to (165.2, 117.2)
Connections:
- C17 pad 1: +3.3V -> +3.3VA
- C18 pad 1: +3.3V -> +3.3VA
- J4 pad 3: GND -> unconnected-(J4-Pin_3-Pad3)
- U3 pad 5: +3.3V -> +3.3VA
- U4 pad 7: +3.3V -> +3.3VA
- U5 pad 1: unconnected-(U5-A0-Pad1) -> GND
- U5 pad 2: unconnected-(U5-A1-Pad2) -> GND
- U5 pad 3: unconnected-(U5-A2-Pad3) -> GND
Routing:
- net +3.3VA: track 5.45 -> 24.0 mm, vias 0 -> 2
- net GND: track 36.0 -> 32.7 mm, vias 31 -> 36
- net +3.3V: track 67.5 -> 65.2 mm, vias 17 -> 14
- net /EEPROM/EEPROM_SCL: track 26.0 -> 27.7 mm, vias 4 -> 1
- net /CAN2.0/Power/NRST: track 63.9 -> 65.4 mm
- net /CAN2.0/Power/3.3IN: track 26.8 -> 25.7 mm
- net Net-(D7-A): track 8.73 -> 9.75 mm
- net +24V Pre: track 26.9 -> 27.9 mm, vias 2 -> 6
- net /EEPROM/EEPROM_SDA: track 31.4 -> 31.0 mm, vias 2 -> 1
Other:
- board text added: "3"
- board text added: "Cain V1.0 Tutor Intel"
- board text added: "David B. 7/25"
