File: PCB_Hardware/Cain/Cain_V1.0/Current_Sense.kicad_sch (KiCad schematic)
At the start: 5 parts, among them U6 INA180A2IDBVR

Commit message: File dump
Parts:
- C22: JLCPCB Part Number (none) -> C1525
- R15: JLCPCB Part Number (none) -> C2988658
- TP3, TP8: now not fitted
- U6: JLCPCB Part Number (none) -> C192764
Other:
- note added: "Current Sensing"
- moved on the sheet: C22, R15, U6
