File: PCB_Hardware/Cain/Cain_V1.0/EEPROM.kicad_sch (KiCad schematic)
At the start: 5 parts, among them J5 Conn_01x04_Pin, U5 24LC01BH

Commit message: File dump
Parts:
- removed U5: 24LC01BH, Package_TO_SOT_SMD:SC-70-8, symbol Memory_EEPROM:24LC01
- added U5: M24C01-RMN, Package_SO:SOIC-8_3.9x4.9mm_P1.27mm, symbol Memory_EEPROM:M24C01-RMN
- C21: JLCPCB Part Number (none) -> C1525
- J5: JLCPCB Part Number (none) -> C37328854
- TP6, TP7: now not fitted
Connections:
- net +3.3V: now also U5.8 (VCC)
- net EEPROM_SCL: now also U5.6 (SCL)
- net EEPROM_SDA: now also U5.5 (SDA)
- net GND: now also U5.1 (E0), U5.2 (E1), U5.3 (E2), U5.4 (VSS), U5.7 (~{WC})
- no-connect marks 3 -> 0
Other:
- note added: "EEPROM"
- moved on the sheet: C21, J5
