File: PCB_Hardware/Cain/Cain_V1.0/MCU.kicad_sch (KiCad schematic)
At the start: 29 parts, among them J1 Conn_ARM_JTAG_SWD_10, J6 Conn_01x04_Pin, SW1 TSB008A2518A, U1 STM32F105RBT6, Y1 X50328MSB2GI (8Mhz)

Commit message: File dump
Parts:
- C1: JLCPCB Part Number (none) -> C19666
- C10, C11: JLCPCB Part Number (none) -> C52923
- C12, C2, C3, C4, C5, C6, C8, C9: JLCPCB Part Number (none) -> C1525
- C7: JLCPCB Part Number (none) -> C15525
- D4: JLCPCB Part Number (none) -> C965834
- D7: JLCPCB Part Number (none) -> C434419
- FB1: JLCPCB Part Number (none) -> C113030
- J1: JLCPCB Part Number (none) -> C2935953
- J6: JLCPCB Part Number (none) -> C37328854
- R1, R16, R2: JLCPCB Part Number (none) -> C25744
- R10, R9: JLCPCB Part Number (none) -> C1211
- R11: JLCPCB Part Number (none) -> C25076
- R14, R17, R6: JLCPCB Part Number (none) -> C4109
- SW1: JLCPCB Part Number (none) -> C2888455
- U1: JLCPCB Part Number (none) -> C8349
- Y1: JLCPCB Part Number (none) -> C115962
Other:
- note added: "MCU"
