File: PCB_Hardware/Cain/Cain_V1.0/Pressure_Sensor.kicad_sch (KiCad schematic)
At the start: 11 parts, among them U3 GZP168-102S, U4 INA333AIDRGR

Commit message: File dump
Parts:
- C17, C18, C19, C20: JLCPCB Part Number (none) -> C1525
- H1, H2: footprint MountingHole:MountingHole_2.7mm_M2.5 -> MountingHole:MountingHole_3.2mm_M3; now not fitted
- R7: JLCPCB Part Number (none) -> C4940
- R8: JLCPCB Part Number (none) -> C11702
- TP1: now not fitted
- U3: JLCPCB Part Number (none) -> C3037990
- U4: JLCPCB Part Number (none) -> C2057429
Connections:
- net +3.3V renamed +3.3VA
Other:
- note added: "Pressure Sensor"
Changed lines of the file:
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@@
+		)
+	)
+	(text "Pressure Sensor"
+		(exclude_from_sim no)
+		(at 79.756 27.178 0)
+		(effects
+			(font
+				(size 10 10)
+				(thickness 1.25)
+			)
 		)
 	)
@@
 			)
 		)
-		(property "JLCPCB Part Number" ""
+		(property "JLCPCB Part Number" "C3037990"
 			(at 119.38 93.98 0)
 			(effects
@@
 		)
 		(property "Sim.Device" ""
+			(at 119.38 93.98 0)
+			(effects
+				(font
+					(size 1.27 1.27)
+				)
+				(hide yes)
+			)
+		)
+		(property "Price" ""
 			(at 119.38 93.98 0)
 			(effects
@@
 		(in_bom no)
 		(on_board yes)
-		(dnp no)
+		(dnp yes)
 		(fields_autoplaced yes)
 		(property "Reference" "TP1"
@@
 		)
 		(property "Sim.Device" ""
+			(at 177.8 93.98 0)
+			(effects
+				(font
+					(size 1.27 1.27)
+				)
+				(hide yes)
+			)
+		)
+		(property "Price" ""
 			(at 177.8 93.98 0)
 			(effects
@@
 		(in_bom no)
 		(on_board yes)
-		(dnp no)
+		(dnp yes)
 		(fields_autoplaced yes)
 		(property "Reference" "H2"
@@
 			)
 		)
-		(property "Footprint" "MountingHole:MountingHole_2.7mm_M2.5"
+		(property "Footprint" "MountingHole:MountingHole_3.2mm_M3"
 			(at 86.36 81.28 0)
 			(effects
@@
 		)
 		(property "Sim.Device" ""
+			(at 86.36 81.28 0)
+			(effects
+				(font
+					(size 1.27 1.27)
+				)
+				(hide yes)
+			)
+		)
+		(property "Price" ""
 			(at 86.36 81.28 0)
 			(effects
@@
 		(in_bom no)
 		(on_board yes)
-		(dnp no)
+		(dnp yes)
 		(fields_autoplaced yes)
 		(property "Reference" "H1"
@@
 			)
 		)
-		(property "Footprint" "MountingHole:MountingHole_2.7mm_M2.5"
+		(property "Footprint" "MountingHole:MountingHole_3.2mm_M3"
 			(at 86.36 76.2 0)
 			(effects
@@
 		)
 		(property "Sim.Device" ""
+			(at 86.36 76.2 0)
+			(effects
+				(font
+					(size 1.27 1.27)
+				)
+				(hide yes)
+			)
+		)
+		(property "Price" ""
 			(at 86.36 76.2 0)
 			(effects
@@
 			)
 		)
-		(property "JLCPCB Part Number" ""
+		(property "JLCPCB Part Number" "C4940"
 			(at 134.62 95.25 0)
 			(effects
@@
 		)
 		(property "Sim.Device" ""
+			(at 134.62 95.25 0)
+			(effects
+				(font
+					(size 1.27 1.27)
+				)
+				(hide yes)
+			)
+		)
+		(property "Price" ""
 			(at 134.62 95.25 0)
 			(effects
@@
 			)
 		)
-		(property "JLCPCB Part Number" ""
+		(property "JLCPCB Part Number" " C11702"
 			(at 166.37 95.25 90)
 			(effects
@@
 		)
 		(property "Sim.Device" ""
+			(at 166.37 95.25 90)
+			(effects
+				(font
+					(size 1.27 1.27)
+				)
+				(hide yes)
+			)
+		)
+		(property "Price" ""
 			(at 166.37 95.25 90)
 			(effects
@@
 			)
 		)
-		(property "Value" "+3.3V"
+		(property "Value" "+3.3VA"
 			(at 119.38 68.58 0)
 			(effects
@@
 			)
 		)
-		(property "Value" "+3.3V"
+		(property "Value" "+3.3VA"
 			(at 151.13 68.58 0)
 			(effects
@@
 			)
 		)
-		(property "JLCPCB Part Number" ""
+		(property "JLCPCB Part Number" " C1525"
 			(at 140.97 80.01 0)
 			(effects
@@
 		)
 		(property "Sim.Device" ""
+			(at 140.97 80.01 0)
+			(effects
+				(font
+					(size 1.27 1.27)
+				)
+				(hide yes)
+			)
+		)
+		(property "Price" ""
 			(at 140.97 80.01 0)
 			(effects
@@
 			)
 		)
-		(property "JLCPCB Part Number" ""
+		(property "JLCPCB Part Number" "C2057429"
 			(at 151.13 95.25 0)
 			(effects
@@
 		)
 		(property "Sim.Device" ""
+			(at 151.13 95.25 0)
+			(effects
+				(font
+					(size 1.27 1.27)
+				)
+				(hide yes)
+			)
+		)
+		(property "Price" ""
 			(at 151.13 95.25 0)
 			(effects
@@
 			)
 		)
-		(property "JLCPCB Part Number" ""
+		(property "JLCPCB Part Number" " C1525"
 			(at 173.99 101.6 0)
 			(effects
@@
 		)
 		(property "Sim.Device" ""
+			(at 173.99 101.6 0)
+			(effects
+				(font
+					(size 1.27 1.27)
+				)
+				(hide yes)
+			)
+		)
+		(property "Price" ""
 			(at 173.99 101.6 0)
 			(effects
@@
 			)
 		)
-		(property "JLCPCB Part Number" ""
+		(property "JLCPCB Part Number" " C1525"
 			(at 109.22 80.01 0)
 			(effects
@@
 		)
 		(property "Sim.Device" ""
+			(at 109.22 80.01 0)
+			(effects
+				(font
+					(size 1.27 1.27)
+				)
+				(hide yes)
+			)
+		)
+		(property "Price" ""
 			(at 109.22 80.01 0)
 			(effects
@@
 			)
 		)
-		(property "JLCPCB Part Number" ""
+		(property "JLCPCB Part Number" " C1525"
 			(at 153.67 107.95 0)
 			(effects
@@
 			(at 153.67 107.95 0)
 			(effects
+				(font
+					(size 1.27 1.27)
+				)
+				(hide yes)
+			)
+		)
+		(property "Price" ""
+			(at 153.67 107.95 0)
+			(effects
