File: PCB_Hardware/Cain/Cain_V1.0/Solenoid.kicad_sch (KiCad schematic)
At the start: 6 parts, among them J2 Conn_01x02_Socket, Q1 STN4NF03L

Commit message: File dump
Parts:
- C16: JLCPCB Part Number (none) -> C1591
- D2: JLCPCB Part Number (none) -> C557917
- J2: JLCPCB Part Number (none) -> C158012
- Q1: JLCPCB Part Number (none) -> C85568
- R4: JLCPCB Part Number (none) -> C25076
- R5: JLCPCB Part Number (none) -> C25741
Other:
- note added: "Solenoid Control"
Changed lines of the file:
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@@
 	(generator_version "9.0")
 	(paper "A4")
+	(text "Solenoid Control"
+		(exclude_from_sim no)
+		(at 80.518 28.194 0)
+		(effects
+			(font
+				(size 10 10)
+				(thickness 1.25)
+			)
+		)
+	)
 	(junction
 		(at 133.35 104.14)
@@
 			)
 		)
-		(property "JLCPCB Part Number" ""
+		(property "JLCPCB Part Number" "C1591"
 			(at 154.94 82.55 0)
 			(effects
@@
 		)
 		(property "Sim.Device" ""
+			(at 154.94 82.55 0)
+			(effects
+				(font
+					(size 1.27 1.27)
+				)
+				(hide yes)
+			)
+		)
+		(property "Price" ""
 			(at 154.94 82.55 0)
 			(effects
@@
 			)
 		)
-		(property "JLCPCB Part Number" ""
+		(property "JLCPCB Part Number" " C158012"
 			(at 170.18 81.28 0)
 			(effects
@@
 		)
 		(property "Sim.Device" ""
+			(at 170.18 81.28 0)
+			(effects
+				(font
+					(size 1.27 1.27)
+				)
+				(hide yes)
+			)
+		)
+		(property "Price" ""
 			(at 170.18 81.28 0)
 			(effects
@@
 			)
 		)
-		(property "JLCPCB Part Number" ""
+		(property "JLCPCB Part Number" " C85568"
 			(at 139.7 93.98 0)
 			(effects
@@
 		)
 		(property "Sim.Device" ""
+			(at 139.7 93.98 0)
+			(effects
+				(font
+					(size 1.27 1.27)
+				)
+				(hide yes)
+			)
+		)
+		(property "Price" ""
 			(at 139.7 93.98 0)
 			(effects
@@
 			)
 		)
-		(property "JLCPCB Part Number" ""
+		(property "JLCPCB Part Number" " C25741"
 			(at 133.35 99.06 0)
 			(effects
@@
 		)
 		(property "Sim.Device" ""
+			(at 133.35 99.06 0)
+			(effects
+				(font
+					(size 1.27 1.27)
+				)
+				(hide yes)
+			)
+		)
+		(property "Price" ""
 			(at 133.35 99.06 0)
 			(effects
@@
 			)
 		)
-		(property "JLCPCB Part Number" ""
+		(property "JLCPCB Part Number" " C557917"
 			(at 142.24 82.55 90)
 			(effects
@@
 		)
 		(property "Sim.Device" ""
+			(at 142.24 82.55 90)
+			(effects
+				(font
+					(size 1.27 1.27)
+				)
+				(hide yes)
+			)
+		)
+		(property "Price" ""
 			(at 142.24 82.55 90)
 			(effects
@@
 			)
 		)
-		(property "JLCPCB Part Number" ""
+		(property "JLCPCB Part Number" "C25076"
 			(at 128.27 93.98 90)
 			(effects
@@
 			(at 128.27 93.98 90)
 			(effects
+				(font
+					(size 1.27 1.27)
+				)
+				(hide yes)
+			)
+		)
+		(property "Price" ""
+			(at 128.27 93.98 90)
+			(effects
