File: PCB_Hardware/Input_Eve/Input_Eve_V1.0/Ethernet.kicad_sch (KiCad schematic)
At the start: 34 parts, among them Q1 WPM2015-3/TR, Q2 LMUN2211LT1G, U2 LAN8710A-EZC, U3 ESDS314DBVR

Commit message: Update w new boards/firmware
Parts:
- removed L1: FB0805/600R/2A, Inductor_SMD:L_0805_2012Metric, symbol Device:L
- removed RJ1: HY931147C, Tutor_Common_Parts:HY931147C, symbol Tutor_Common_Parts:HY931147C
- added C110, C27, C28, C29: 1000p, 2kV, Capacitor_SMD:C_0402_1005Metric, symbol Device:C
- added C25, C26: 18p, Capacitor_SMD:C_0402_1005Metric, symbol Device:C
- added C30, C31: 4.7n, Capacitor_SMD:C_0402_1005Metric, symbol Device:C
- added FB2: FB0805/600R/2A, Inductor_SMD:L_0603_1608Metric, symbol Device:FerriteBead
- added J5: 0826-1X1T-HS-F, Tutor_Common_Parts:CONN_0826-1X1T-HS-F_BEL, symbol Tutor_Common_Parts:0826-1X1T-HS-F
- added R22, R23, R24, R25: 75, Resistor_SMD:R_0402_1005Metric, symbol Device:R
- added R26, R27, R28, R29: 49.9, Resistor_SMD:R_0402_1005Metric, symbol Device:R
- added R91: 10k, Resistor_SMD:R_0402_1005Metric, symbol Device:R
- added Y1: XXGBBCNANF-25.000000MHZ, Crystal:Crystal_SMD_3225-4Pin_3.2x2.5mm, symbol Device:Crystal_GND24
- C15: renamed from C12; footprint Capacitor_SMD:C_0603_1608Metric -> Capacitor_SMD:C_0402_1005Metric
- C16: renamed from C13; footprint Capacitor_SMD:C_0603_1608Metric -> Capacitor_SMD:C_0402_1005Metric
- C17: renamed from C15; footprint Capacitor_SMD:C_0603_1608Metric -> Capacitor_SMD:C_0402_1005Metric
- C22: renamed from C19; footprint Capacitor_SMD:C_0603_1608Metric -> Capacitor_SMD:C_0402_1005Metric
- R13: renamed from R10; value 2.2k -> 10k
- R14: renamed from R11; value 2.2k -> 10k
- R17: renamed from R12; value 2.2k -> 10k
- R18: renamed from R13; value 2.2k -> 10k
- R19: renamed from R15; value 2.2k -> 10k
- R4: renamed from R2; footprint (none) -> Resistor_SMD:R_0402_1005Metric
- renumbered C16 to C18, C17 to C19, C18 to C20, C14 to C21, C20 to C23, C21 to C24, R8 to R10, R9 to R11, R17 to R12, R18 to R15, R14 to R16, R16 to R20, R19 to R21, R4 to R5, R5 to R6, R6 to R7, R7 to R8, R3 to R9, U3 to U2, U2 to U3
Connections:
- net +3.3VLAN: now also FB2.1, R91.2
- net ETHGREEN: now also J5.20 (LED3)
- net ETHYELLOW: now also J5.18 (LED1)
- net ETH_REF_CLK: now also C25.1, Y1.1
- net GND: now also Q2.2 (E), R12.1, C110.1, C25.2, C26.2, C27.1, C28.1, C29.1, C30.2, C31.2, Y1.2, Y1.4; no longer Q2.E
- net PHY_PWR: now also Q2.1 (B); no longer Q2.B
- net at C17.1, C18.1, C19.1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: now also FB2.2; no longer R12.2
- net at R9.2: now also Q2.3 (C); no longer Q2.C
- net at R5.2, U2.3 (I/O2), U3.29 (TXP): now also J5.4 (TRD2+)
- net at R6.2, U2.4 (I/O3), U3.28 (TXN): now also J5.5 (TRD2-)
- net at R8.2, U2.5 (I/O4), U3.30 (RXN): now also J5.10 (TRD1-)
- net ETH_INT: now reaches U3.18 (~{INT}/TXER/TXD4)
- net ETH_INT: now also R91.1
- net at R7.2, U2.1 (I/O1), U3.31 (RXP): now also J5.11 (TRD1+)
- net at U3.4 (XTAL2): now also C26.1, Y1.3
- net at R15.1: now also J5.17 (LED1)
- net ETH_RXD0 renamed ETH_RXD+
- net ETH_RXD1 renamed ETH_RXD-
- net ETH_TXD0 renamed ETH_TXD+
- net ETH_TXD1 renamed ETH_TXD-
- new net: C30.1, C31.1, J5.21 (SHIELD), J5.22 (SHIELD)
- new net: J5.19 (LED2), R12.2
- new net: C28.2, C29.2, R26.2, R27.2, R28.2, R29.2
- new net: J5.1 (TRCT3), R23.1
- new net: C110.2, C27.2, R22.2, R23.2, R24.2, R25.2
- new net: J5.2 (TRD3-), R28.1
- new net: J5.6 (TRCT2), R24.1
- new net: J5.7 (TRCT4), R22.1
- new net: J5.8 (TRD4+), R27.1
- new net: J5.12 (TRCT1), R25.1
- new net: J5.3 (TRD3+), R29.1
- new net: J5.9 (TRD4-), R26.1
- new net VC1: J5.13 (VC1)
- new net VC2: J5.14 (VC2)
- new net VC3: J5.15 (VC3)
- new net VC4: J5.16 (VC4)
- no-connect marks 5 -> 3
Other:
- moved on the sheet: C15, C16, C17, C18, C19, C20, C21, C22, C23, C24, Q1, Q2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
