File: PCB_Hardware/Input_Eve/Input_Eve_V1.0/Input_Eve_V1.0.kicad_sch (KiCad schematic)
At the start: 0 parts

Commit message: Update w new boards/firmware
Parts:
- added H1, H2, H3, H4: MountingHole, MountingHole:MountingHole_3.2mm_M3, symbol Mechanical:MountingHole
Other:
- sheet USB renamed USB (Flash)
- added sheet Estop (Estop.kicad_sch)
- added sheet FRAM (untitled.kicad_sch)
- added sheet Fans (Enclosure_Fans.kicad_sch)
- added sheet Hall Effects (Hall_Effects.kicad_sch)
- added sheet IMU (IMU.kicad_sch)
- added sheet Input Current Sense (Current Sense.kicad_sch)
- added sheet LEDs (LEDs.kicad_sch)
- added sheet MIC (MIC.kicad_sch)
- added sheet Output Current Sense (Output_Current_Sense.kicad_sch)
- added sheet QSPI Flash (QSPI_Flash.kicad_sch)
- added sheet Relay Control (Relay_Control.kicad_sch)
- added sheet Temp Sensor (Temp_Sensor.kicad_sch)
- added sheet Temp Sensors (Temp_Sensors.kicad_sch)
- added sheet USB_Host (External_Temp_Sensor.kicad_sch)
- sheet Ethernet ports: added ETH_CRS_DV, ETH_INT, ETH_MDC, ETH_MDIO, ETH_REF_CLK, ETH_RXD+, ETH_RXD-, ETH_TXD+, ETH_TXD-, ETH_TX_EN, PHY_PWR, VC1, VC2, VC3, VC4; removed none
- sheet External Sensors ports: added +24_Post_1, +24_Post_10, +24_Post_2, +24_Post_3, +24_Post_4, +24_Post_5, +24_Post_6, +24_Post_7, +24_Post_8, +24_Post_9, R1IN, R2IN, RS485+, RS485-, T1OUT, T2OUT; removed none
- sheet MCU ports: added BT, Board_Fan_FG, Board_Fan_Tim, Board_Monitor_SCL, Board_Monitor_SDA, CS, CS_IMU, DFSDM_CLK, DFSDM_DATA, ETH_CRS_DV, ETH_INT, ETH_MDC, ETH_MDIO, ETH_REF_CLK, ETH_RXD+, ETH_RXD-, ETH_TXD+, ETH_TXD-, ETH_TX_EN, Fan_1, Fan_2, Fan_3, Fan_4, Fan_5, Fan_6, Fan_Curr_1, Fan_Curr_2, Fan_Curr_3, Fan_Curr_4, Fan_Curr_5, Fan_Curr_6, Fan_FG_1, Fan_FG_2, Fan_FG_3, Fan_FG_4, Fan_FG_5, Fan_FG_6, Flash_CS, Flash_IO0, Flash_IO1, Flash_IO2, Flash_IO3, Flash_SPI_CLK, HALL_1, HALL_10, HALL_2, HALL_3, HALL_4, HALL_5, HALL_6, HALL_7, HALL_8, HALL_9, HOLD, IMU_INT_1, IMU_INT_2, Input_Curr_INT, LED_Control, MISO, MOSI, PHY_PWR, RS232_RX_1, RS232_RX_2, RS232_TX_1, RS232_TX_2, RS485_DE, RS485_RX, RS485_TX, SCK, SEL, Sensor_Curr_1, Sensor_Curr_10, Sensor_Curr_2, Sensor_Curr_3, Sensor_Curr_4, Sensor_Curr_5, Sensor_Curr_6, Sensor_Curr_7, Sensor_Curr_8, Sensor_Curr_9, TEMP_USB_D+, TEMP_USB_D-, TEMP_USB_VBUS, TPH, TPL, Temp_ALERT, Temp_Sense_1, Temp_Sense_2, Temp_Sense_3, Temp_Sense_4, USB_D+, USB_D-, USB_EN, USB_Fault, USB_VBUS; removed none
- sheet POE ports: added 24V Pre, BT, TPH, TPL, VC1, VC2, VC3, VC4; removed none
- sheet RS232 ports: added R1IN, R2IN, RS232_RX_1, RS232_RX_2, RS232_TX_1, RS232_TX_2, T1OUT, T2OUT; removed none
- sheet RS485 ports: added RS485+, RS485-, RS485_DE, RS485_RX, RS485_TX; removed none
- sheet USB (Flash) ports: added USB_D+, USB_D-, USB_VBUS; removed none
