File: PCB_Hardware/Input_Eve/Input_Eve_V1.0/Power.kicad_sch (KiCad schematic)
At the start: 0 parts

Commit message: Update w new boards/firmware
Parts:
- added C42, C43: 22u, Capacitor_SMD:C_0402_1005Metric, symbol Device:C
- added C57: 10u, Capacitor_SMD:C_0402_1005Metric, symbol Device:C
- added C58, C59, C89, C90: 100n, Capacitor_SMD:C_0402_1005Metric, symbol Device:C
- added C60, C61, C62: 22u, Capacitor_SMD:C_0603_1608Metric, symbol Device:C
- added C80, C81, C82, C83: 4.7u, Capacitor_SMD:C_1210_3225Metric, symbol Device:C
- added C84, C85, C86, C87: 22u, Capacitor_SMD:C_1206_3216Metric, symbol Device:C
- added C88: 2.2u, Capacitor_SMD:C_0402_1005Metric, symbol Device:C
- added C91: 6.8u, Capacitor_SMD:C_0402_1005Metric, symbol Device:C
- added C92: 100p, Capacitor_SMD:C_0402_1005Metric, symbol Device:C
- added D19, D39: LED, LED_SMD:LED_0603_1608Metric, symbol Device:LED
- added D6: RED, Diode_SMD:D_0603_1608Metric, symbol Device:D
- added L1: 15u, Tutor_Common_Parts:IND_CYA0630_SHH, symbol Device:L
- added L2: 6.8uH, Inductor_SMD:L_Vishay_IHLP-4040, symbol Device:L
- added Q12, Q13: Q_NMOS, Package_TO_SOT_SMD:TDSON-8-1, symbol Device:Q_NMOS
- added R34: R, Resistor_SMD:R_0402_1005Metric, symbol Device:R
- added R61: 511k, Resistor_SMD:R_0402_1005Metric, symbol Device:R
- added R62: 105k, Resistor_SMD:R_0402_1005Metric, symbol Device:R
- added R63: 49.9, Resistor_SMD:R_0402_1005Metric, symbol Device:R
- added R64: 100k, Resistor_SMD:R_0402_1005Metric, symbol Device:R
- added R65: 13.3k, Resistor_SMD:R_0402_1005Metric, symbol Device:R
- added R66, R86: 2.2k, Resistor_SMD:R_0402_1005Metric, symbol Device:R
- added R81: 5m, Resistor_SMD:R_1206_3216Metric, symbol Device:R
- added R82, R83: 48.7k, Resistor_SMD:R_0402_1005Metric, symbol Device:R
- added R84: 41.2k, Resistor_SMD:R_0402_1005Metric, symbol Device:R
- added R85: 4.75, Resistor_SMD:R_0402_1005Metric, symbol Device:R
- added U14: TPS54202DDC, Package_TO_SOT_SMD:SOT-23-6, symbol Regulator_Switching:TPS54202DDC
- added U17: LM5148RGYR, Tutor_Common_Parts:QFN50P550X350X100-25N, symbol Tutor_Common_Parts:LM5148RGYR
- added U8: AMS1117-3.3, Package_TO_SOT_SMD:SOT-223-3_TabPin2, symbol Regulator_Linear:AMS1117-3.3
Connections:
- new net: C91.1, R85.2
- new net: C59.2, L1.1, U14.2 (SW)
- new net: C90.1, U17.15 (CBOOT)
- new net: C90.2, L2.1, Q12.1 (S), Q12.2 (S), Q12.3 (S), Q13.5 (D), U17.14 (SW)
- new net: R82.2, U17.6 (FB)
- new net: D39.1 (K), R86.1
- new net: C59.1, U14.6 (BOOT)
- new net: R61.2, R62.1, U14.5 (EN)
- new net: D19.1 (K), R66.1
- new net: C62.1, R63.2, R64.1
- new net: D6.1 (K), R34.1
- new net: C62.2, R64.2, R65.1, U14.4 (FB)
- new net: R83.2, U17.4 (RT)
- new net: C88.1, U17.9 (VCC)
- new net: R84.2, U17.3 (CNFG)
- new net: C92.1, R85.1, U17.5 (EXTCOMP)
- new net: Q13.4 (G), U17.11 (LO)
- new net: Q12.4 (G), U17.13 (HO)
- new net: L2.2, R81.1, U17.20 (ISNS+)
- new net +12V: C84.1, C85.1, C86.1, C87.1, D39.2 (A), R81.2, U17.21 (VOUT)
- new net +24V: C57.1, C58.1, C80.1, C81.1, C82.1, C83.1, Q12.5 (D), R61.1, U14.3 (VIN), U17.12 (VIN), U17.19 (EN)
- new net +3.3V: C43.1, D6.2 (A), U8.2 (VO)
- new net +5V: C42.1, C60.1, C61.1, D19.2 (A), L1.2, R63.1, U8.3 (VI)
- new net GND: C42.2, C43.2, C57.2, C58.2, C60.2, C61.2, C80.2, C81.2, C82.2, C83.2, C84.2, C85.2, C86.2, C87.2, C88.2, C89.2, C91.2, C92.2, Q13.1 (S), Q13.2 (S), Q13.3 (S), R34.2, R62.2, R65.2, R66.2, R83.1, R84.1, R86.2, U14.1 (GND), U17.10 (PGND), U17.16 (VCCX), U17.25 (EP), U17.7 (AGND), U8.1 (GND)
- new net VDDA: C89.1, R82.1, U17.8 (VDDA)
- no-connect marks 0 -> 2
Other:
- note added: "IAUC28N08S5L230ATMA1"
- note added: "IHLP4040DZER6R8M8A"
- note added: "SHOU HAN CYA0630-15UH"
