File: PCB_Hardware/Input_Eve/Input_Eve_V1.0/RS425.kicad_sch (KiCad schematic)
At the start: 7 parts, among them U8 MAX485ESA+T

Commit message: Update w new boards/firmware
Parts:
- added J35, J37: Conn_01x02_Socket, Connector_JST:JST_PH_B2B-PH-K_1x02_P2.00mm_Vertical, symbol Connector:Conn_01x02_Socket
- added R71: 120, Resistor_SMD:R_0402_1005Metric, symbol Device:R
- C44: renamed from C29; value 0.1u -> 100n
- renumbered R39 to R36, R41 to R37, R42 to R38, R43 to R39, U8 to U9
Connections:
- net RS485+: now also J35.1 (Pin_1)
- net RS485-: now also J35.2 (Pin_2)
- new net Term+: J37.1 (Pin_1), R71.1
- new net Term-: J37.2 (Pin_2), R71.2
