File: PCB_Hardware/Input_Eve/Input_Eve_V1.0/Sensors.kicad_sch (KiCad schematic)
At the start: 9 parts, among them J3 Conn_01x04_Socket, J3 Conn_01x05_Socket

Commit message: Update w new boards/firmware
Parts:
- removed D10, D18: SM712_SOT23, Package_TO_SOT_SMD:SOT-23, symbol Diode:SM712_SOT23
- removed J3: Conn_01x05_Socket, symbol Connector:Conn_01x05_Socket
- removed J3: Conn_01x04_Socket, symbol Connector:Conn_01x04_Socket
- added C109, C120, C122, C124, C125, C47, C48, C49: 100n, Capacitor_SMD:C_0402_1005Metric, symbol Device:C
- added D20, D21, D22, D23: SMBJ12CA, Diode_SMD:D_SMA, symbol Diode:SMAJ6.0CA
- added J10, J12, J2, J7, J8, J9: Conn_01x02_Socket, Connector_Molex:Molex_Micro-Latch_53253-0270_1x02_P2.00mm_Vertical, symbol Connector:Conn_01x02_Socket
- added J13: DE9_Socket_MountingHoles, Connector_Dsub:DSUB-9_Socket_Horizontal_P2.77x2.84mm_EdgePinOffset4.94mm_Housed_MountingHolesOffset4.94mm, symbol Connector:DE9_Socket_MountingHoles
- added J27, J6: Conn_01x04_Socket, Connector_Molex:Molex_Micro-Fit_3.0_43650-0400_1x04_P3.00mm_Horizontal, symbol Connector:Conn_01x04_Socket
- added J34, J36: Conn_01x02_Socket, Connector_JST:JST_PH_B2B-PH-K_1x02_P2.00mm_Vertical, symbol Connector:Conn_01x02_Socket
- renumbered C33 to C45, C35 to C46, D11 to D8, D12 to D9, R44 to R41
Connections:
- net GND: now also C109.2, C120.2, C122.2, C124.2, C125.2, C47.2, C48.2, C49.2, D20.1 (A1), D21.1 (A1), D22.1 (A1), D23.1 (A1), J10.1 (Pin_1), J12.1 (Pin_1), J13.5, J2.1 (Pin_1), J27.1 (Pin_1), J34.1 (Pin_1), J36.1 (Pin_1), J6.1 (Pin_1), J7.1 (Pin_1), J8.1 (Pin_1), J9.1 (Pin_1)
- net at D9.1 (K): now also D8.1 (K)
- net at D9.2 (A): now also J6.2 (Pin_2); no longer D8.1 (K)
- net +24V renamed +24_Post_2
- net +24_Post_2: now also J2.2 (Pin_2); no longer C45.1
- new net +24_Post_1: C48.1, J8.2 (Pin_2)
- new net +24_Post_10: C109.1, J27.4 (Pin_4)
- new net +24_Post_3: C47.1, J7.2 (Pin_2)
- new net +24_Post_4: C49.1, J9.2 (Pin_2)
- new net +24_Post_5: C122.1, J12.2 (Pin_2)
- new net +24_Post_6: C120.1, J10.2 (Pin_2)
- new net +24_Post_7: C125.1, J36.2 (Pin_2)
- new net +24_Post_8: C124.1, J34.2 (Pin_2)
- new net +24_Post_9: C45.1, J6.4 (Pin_4)
- new net R1IN: D20.2 (A2), J13.2
- new net R2IN: D23.2 (A2), J27.2 (Pin_2)
- new net T1OUT: D21.2 (A2), J13.3
- new net T2OUT: D22.2 (A2), J27.3 (Pin_3)
- no-connect marks 0 -> 1
Other:
- note added: "AUX1 24V"
- note added: "AUX2 24V"
- note added: "AUX3 24V"
- note added: "AUX4 24V"
- note added: "Designed to be used with the FM350-6000RG112K"
- note added: "Flow Sense"
- note added: "UPS"
- moved on the sheet: C45
