File: PCB_Hardware/Input_Eve/Input_Eve_V1.0/USB.kicad_sch (KiCad schematic)
At the start: 3 parts, among them J2 USB_B

Commit message: Update w new boards/firmware
Parts:
- added C41: 100n, Capacitor_SMD:C_0402_1005Metric, symbol Device:C
- added D5: SMBJ5.0A, Diode_SMD:D_SMB, symbol Device:D_Zener
- added U7: USBLC6-2SC6, Package_TO_SOT_SMD:SOT-23-6, symbol Power_Protection:USBLC6-2SC6
- D4: renamed from D3; value LED -> RED; footprint (none) -> LED_SMD:LED_0603_1608Metric
- J4: renamed from J2; value USB_B -> 5787834
- R33: renamed from R30; footprint (none) -> Resistor_SMD:R_0402_1005Metric
Connections:
- net +5V USB: now also C41.1, D5.1 (K), U7.5 (VBUS)
- net GND: now also C41.2, D5.2 (A), U7.2 (GND)
- net USB_D+: now also U7.6 (I/O1); no longer J4.3 (D+)
- net USB_D-: now also U7.4 (I/O2); no longer J4.2 (D-)
- new net D+: J4.3 (D+), U7.1 (I/O1)
- new net D-: J4.2 (D-), U7.3 (I/O2)
Other:
- moved on the sheet: D4, J4, R33
